File: pcb/lo_cate_pcb/lo_cate_pcb.kicad_pcb (KiCad board)
At the start: 4 copper layers, 100 x 50 mm, 58 parts, among them J1 Conn_01x07_Pin, J2 690-005-299-043, SW1 MICRO_RESET, SW2 MICRO_ON, SW3 BUTTON1, SW4 BUTTON2, SW5 BUTTON3, U1 STM32F401RETx, U2 BMI323, U3 LED1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

Commit message: Moved the Oscillator slightly to help with assembly
Parts:
- moved C18 1.76 mm to (220.1, 134.1)
- moved Y1 1.45 mm to (220.1, 128.0)
Routing:
- net Net-(C19-Pad1): track 9.63 -> 10.5 mm
- net /OSC_IN: track 20.7 -> 20.1 mm
Changed lines of the file:
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@@
 	(footprint "Crystal:Crystal_SMD_7050-4Pin_7.0x5.0mm"
 		(layer "F.Cu")
-		(at 221.5 127.5 90)
+		(at 220.125 127.975 90)
 		(descr "SMD Crystal SERIES SMD7050/4 https://www.foxonline.com/pdfs/FQ7050.pdf, 7.0x5.0mm^2 package")
 		(tags "SMD SMT crystal")
@@
 	(footprint "Capacitor_SMD:C_0805_2012Metric_Pad1.18x1.45mm_HandSolder"
 		(layer "F.Cu")
-		(at 221.5 133 180)
+		(at 220.125 134.1 180)
 		(descr "Capacitor SMD 0805 (2012 Metric), square (rectangular) end terminal, IPC_7351 nominal with elongated pad for handsoldering. (Body size source: IPC-SM-782 page 76, https://www.pcb-3d.com/wordpress/wp-content/uploads/ipc-sm-782a_amendment_1_and_2.pdf, https://docs.google.com/spreadsheets/d/1BsfQQcO9C6DZCsRaXUlFlo91Tg2WpOkGARC1WS5S8t0/edit?usp=sharing), generated with kicad-footprint-generator")
 		(tags "capacitor handsolder")
@@
 	)
 	(segment
-		(start 222.5375 130.7625)
-		(end 222.85 130.45)
+		(start 221.475 133.7875)
+		(end 221.1625 134.1)
 		(width 0.2)
 		(layer "F.Cu")
@@
 	)
 	(segment
-		(start 213 123.5)
-		(end 210.75 121.25)
+		(start 221.475 130.925)
+		(end 221.475 133.7875)
 		(width 0.2)
 		(layer "F.Cu")
@@
 	)
 	(segment
-		(start 222.85 130.45)
-		(end 217.4 125)
+		(start 213 123.5)
+		(end 210.75 121.25)
 		(width 0.2)
 		(layer "F.Cu")
@@
 	)
 	(segment
-		(start 222.5375 133)
-		(end 222.5375 130.7625)
+		(start 215.425 125.925)
+		(end 216.475 125.925)
 		(width 0.2)
 		(layer "F.Cu")
@@
 	)
 	(segment
-		(start 217.4 125)
-		(end 216 125)
+		(start 216.475 125.925)
+		(end 221.475 130.925)
 		(width 0.2)
 		(layer "F.Cu")
@@
 	)
 	(via
-		(at 216 125)
+		(at 215.425 125.925)
 		(size 0.6)
 		(drill 0.3)
@@
 	)
 	(segment
-		(start 214.5 125)
+		(start 215.425 125.925)
 		(end 213 123.5)
 		(width 0.2)
@@
 	)
 	(segment
-		(start 216 125)
-		(end 214.5 125)
-		(width 0.2)
-		(layer "B.Cu")
-		(net 44)
-	)
-	(segment
 		(start 196.550001 105.699999)
 		(end 196.75 105.5)
@@
 	)
 	(segment
-		(start 214 120.5)
-		(end 215.5 120.5)
+		(start 218.775 125.025)
+		(end 218.775 123.1875)
 		(width 0.2)
 		(layer "F.Cu")
@@
 	)
 	(segment
-		(start 219.9625 122)
-		(end 219.9625 124.3625)
+		(start 218.775 123.1875)
+		(end 219.9625 122)
 		(width 0.2)
 		(layer "F.Cu")
@@
 	)
 	(segment
-		(start 219.9625 124.3625)
-		(end 220.15 124.55)
+		(start 214 120.5)
+		(end 215.5 120.5)
 		(width 0.2)
 		(layer "F.Cu")

Commit message: Altered the Oscillator Path
Parts:
- moved C10 64.6 mm to (145.8, 82.8)
- moved J1 64.6 mm to (167.2, 77.6)
- moved C7 64.6 mm to (124.4, 80.3)
- moved C8 64.6 mm to (124.4, 83.8)
- moved J2 64.6 mm to (102.8, 82.2)
- moved C1 64.6 mm to (151.5, 112.8)
- moved C11 64.6 mm to (146.6, 104.8)
- moved C12 64.6 mm to (134.5, 101.1)
- moved C13 64.6 mm to (135.8, 87.5)
- moved C14 64.6 mm to (155.2, 90.8)
- moved C15 64.6 mm to (139.0, 85.6)
- moved C18 64.6 mm to (160.2, 110.2)
- moved C19 64.6 mm to (161.0, 98.1)
- moved C2 64.6 mm to (165.0, 112.1)
- moved C3 64.6 mm to (192.0, 107.1)
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Routing:
- net /OSC_IN: track 20.1 -> 24.1 mm
- net GND: vias 3 -> 6
